File: r2/midi-thru.kicad_pcb (KiCad board)
At the start: 2 copper layers, 75 x 70 mm, 33 parts, among them J1 Barrel_Jack_Switch, J2 MIDI IN, J4 MIDI THRU3, J5 MIDI THRU1, J6 MIDI THRU2, J7 MIDI THRU3, U2 6N138, U3 74HC14

Commit message: Add voltage regulator
Parts:
- added C3: 10 uF, Capacitor_THT:CP_Radial_D5.0mm_P2.00mm, F.Cu at (38.5, 85.4)
- added C4: 100 nF, Capacitor_THT:C_Disc_D5.0mm_W2.5mm_P5.00mm, F.Cu at (37.7, 81.1)
- added Q1: IRLZ44N, Package_TO_SOT_THT:TO-220-3_Vertical, F.Cu at (28.8, 80.8)
- added R7: 15K, Resistor_THT:R_Axial_DIN0204_L3.6mm_D1.6mm_P7.62mm_Horizontal, F.Cu at (37.6, 78.5)
- added U1: L7805, Package_TO_SOT_THT:TO-220-3_Vertical, F.Cu at (28.8, 85.8)
- C2: footprint Capacitor_THT:CP_Radial_D5.0mm_P2.50mm -> Capacitor_THT:CP_Radial_D5.0mm_P2.00mm
- D1: value UF4007 -> D_Zener; footprint Diode_THT:D_DO-41_SOD81_P10.16mm_Horizontal -> Diode_THT:D_DO-35_SOD27_P7.62mm_Horizontal
- D3: value RED -> MIDI ACT
- moved J4 54.7 mm to (127.6, 110.7), turned to 0 degrees
Connections:
- C1 pad 1: VCC -> Net-(C1-Pad1)
- C1 pad 2: GND -> Net-(C1-Pad2)
- C2 pad 1: VCC -> Net-(C1-Pad1)
- D1 pad 1: VCC -> Net-(C1-Pad2)
- D1 pad 2: Net-(D1-Pad2) -> GND
- J1 pad 1: Net-(D1-Pad2) -> Net-(C1-Pad1)
- J1 pad 2: GND -> Net-(J1-Pad2)
- J1 pad 3: GND -> Net-(J1-Pad2)
- R14 pad 1: VCC -> Net-(C1-Pad1)

Commit message: Update PDF schematics
Parts:
- removed D6: PWR, LED_THT:LED_D5.0mm
- removed J7: MIDI THRU3, turnandpush:din-5
- added D4: MIDI ACT, LED_THT:LED_D5.0mm, F.Cu at (114.7, 76.1)
- added J3: MIDI THRU1, turnandpush:din-5, F.Cu at (68.9, 106.0)
- C2, C3: value 10 uF -> 100 uF; footprint Capacitor_THT:CP_Radial_D5.0mm_P2.00mm -> Capacitor_THT:CP_Radial_D6.3mm_P2.50mm
- D1: value D_Zener -> 1N4148
- D2: value 1N4148 -> D_Zener
- D3: value MIDI ACT -> PWR
- J4: value MIDI THRU3 -> MIDI THRU2
- J5: value MIDI THRU1 -> MIDI THRU3
- J6: value MIDI THRU2 -> MIDI THRU4
- R1: value 220 -> 15K
- R2: value 330 -> 220
- R3: value 220 -> 330
- R7: value 15K -> 220
- U1: value L7805 -> 6N138; footprint Package_TO_SOT_THT:TO-220-3_Vertical -> Package_DIP:DIP-8_W7.62mm_Socket
- U2: value 6N138 -> L7805; footprint Package_DIP:DIP-8_W7.62mm_Socket -> Package_TO_SOT_THT:TO-220-3_Vertical
- moved LOGO_OSHW_silkscreen_5mm 102.3 mm to (223.2, 66.4)
- moved U1 97.7 mm to (126.5, 83.3), turned to 270 degrees
- moved D1 74.8 mm to (133.8, 91.0)
- moved C4 74.1 mm to (109.4, 62.1), turned to 270 degrees
- moved C3 70.6 mm to (108.0, 73.1), turned to 270 degrees
- moved Q1 52.1 mm to (80.3, 73.1), turned to 180 degrees
- moved R2 51.4 mm to (130.3, 90.8), turned to 90 degrees
- moved R14 51.1 mm to (114.5, 61.1), turned to 270 degrees
- moved R3 51.0 mm to (65.9, 84.0)
- moved R5 44.9 mm to (113.2, 91.2), turned to 90 degrees
- moved J2 42.9 mm to (129.9, 66.3)
- moved J6 41.2 mm to (128.4, 106.0)
- moved J4 39.1 mm to (88.8, 106.0)
- moved R7 34.4 mm to (71.7, 83.2), turned to 270 degrees
- moved U3 33.6 mm to (92.7, 90.8)
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Connections:
- D1 pad 1: Net-(C1-Pad2) -> Net-(D1-Pad1)
- D1 pad 2: GND -> Net-(D1-Pad2)
- D2 pad 1: Net-(D2-Pad1) -> Net-(C1-Pad2)
- D2 pad 2: Net-(D2-Pad2) -> GND
- D3 pad 1: Net-(D3-Pad1) -> GND
- D3 pad 2: VCC -> Net-(D3-Pad2)
- J2 pad 5: Net-(D2-Pad2) -> Net-(D1-Pad2)
- R1 pad 1: Net-(D2-Pad1) -> Net-(C1-Pad1)
- R1 pad 2: Net-(J2-Pad4) -> Net-(C1-Pad2)
- R10 pad 2: Net-(J6-Pad5) -> Net-(J5-Pad5)
- R11 pad 2: Net-(J6-Pad4) -> Net-(J5-Pad4)
- R12 pad 2: Net-(J7-Pad5) -> Net-(J6-Pad5)
- R13 pad 2: Net-(J7-Pad4) -> Net-(J6-Pad4)
- R14 pad 1: Net-(C1-Pad1) -> Net-(D4-Pad1)
- R14 pad 2: Net-(D6-Pad2) -> Net-(R14-Pad2)
- R2 pad 1: Net-(D3-Pad1) -> Net-(D1-Pad1)
- R2 pad 2: Net-(R2-Pad2) -> Net-(J2-Pad4)
- R3 pad 1: Net-(R3-Pad1) -> Net-(C1-Pad1)
- R3 pad 2: Net-(J4-Pad5) -> Net-(D3-Pad2)
- R6 pad 1: VCC -> Net-(R6-Pad1)
- R6 pad 2: Net-(J4-Pad4) -> Net-(J3-Pad5)
- R7 pad 1: Net-(C1-Pad1) -> VCC
- R7 pad 2: Net-(C1-Pad2) -> Net-(J3-Pad4)
- R8 pad 2: Net-(J5-Pad5) -> Net-(J4-Pad5)
- R9 pad 2: Net-(J5-Pad4) -> Net-(J4-Pad4)
- U1 pad 1: Net-(C1-Pad1) -> Net-(U1-Pad1)
- U1 pad 2: GND -> Net-(D1-Pad1)
- U1 pad 3: VCC -> Net-(D1-Pad2)
- U2 pad 1: Net-(U2-Pad1) -> Net-(C1-Pad1)
- U2 pad 2: Net-(D2-Pad1) -> GND
- U2 pad 3: Net-(D2-Pad2) -> VCC
- U3 pad 10: Net-(R3-Pad1) -> Net-(R12-Pad1)
- U3 pad 12: Net-(R2-Pad2) -> Net-(R14-Pad2)
- U3 pad 4: Net-(R8-Pad1) -> Net-(R6-Pad1)
- U3 pad 6: Net-(R10-Pad1) -> Net-(R8-Pad1)
- U3 pad 8: Net-(R12-Pad1) -> Net-(R10-Pad1)
Other:
- board size 75 x 70 mm -> 100.2 x 70.5 mm
